Commit message: minor fix: removed joint_state_publisher from static display

File: anrobot_description/urdf/static.urdf (robot description, URDF)
Before this commit: robot test_robot, 7 links, 6 joints
Joints:
- joint joint1: axis 0 0 1 -> (none); type continuous -> fixed
- joint joint2: axis 0 0 1 -> (none); type continuous -> fixed
- joint joint3: axis 0 0 1 -> (none); type continuous -> fixed
